File: hw/sch_pcb/RFIQINT02A.kicad_sch (KiCad schematic)
At the start: 33 parts, among them J1 HEADER_2x03_PARALLEL, J2 HEADER_2x04_PARALLEL, J3 SATA7-67491-1030, J4 SATA7-67491-1030, J5 SATA7-67491-1030, J6 RJ45_RJHSE-5384, J7 RJ45_RJHSE-5384, M1 HOLE, M2 HOLE, M3 HOLE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

Commit message: Edit PCB
Connections:
- net CLKOUT0_N: now also C9.2; no longer C7.2
- net CLKOUT0_P: now also C8.2; no longer C6.2
- net CLKOUT1_N: now also C7.2; no longer C9.2
- net CLKOUT1_P: now also C6.2; no longer C8.2
Changed lines of the file:
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@@
   (junction (at 262.89 149.86) (diameter 0) (color 0 0 0 0))
   (junction (at 268.605 149.86) (diameter 0) (color 0 0 0 0))
+  (no_connect (at 45.72 64.77))
   (no_connect (at 45.72 67.31))
-  (no_connect (at 45.72 64.77))
   (wire (pts (xy 27.94 144.78) (xy 29.845 144.78))
     (stroke (width 0) (type solid) (color 0 0 0 0))
@@
     (stroke (width 0) (type solid) (color 0 0 0 0))
   )
-  (label "CLKOUT0_P" (at 160.02 61.595 0)
+  (label "CLKOUT1_P" (at 160.02 61.595 0)
     (effects (font (size 1.524 1.524)) (justify left bottom))
   )
-  (label "CLKOUT0_N" (at 160.02 67.31 0)
+  (label "CLKOUT1_N" (at 160.02 67.31 0)
     (effects (font (size 1.524 1.524)) (justify left bottom))
   )
-  (label "CLKOUT1_P" (at 160.02 72.39 0)
+  (label "CLKOUT0_P" (at 160.02 72.39 0)
     (effects (font (size 1.524 1.524)) (justify left bottom))
   )
-  (label "CLKOUT1_N" (at 160.02 77.47 0)
+  (label "CLKOUT0_N" (at 160.02 77.47 0)
     (effects (font (size 1.524 1.524)) (justify left bottom))
   )

Commit message: Edit PCB
Connections:
- net GND: now also M4.1
Changed lines of the file:
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@@
   (junction (at 262.89 149.86) (diameter 0) (color 0 0 0 0))
   (junction (at 268.605 149.86) (diameter 0) (color 0 0 0 0))
+  (no_connect (at 45.72 67.31))
   (no_connect (at 45.72 64.77))
-  (no_connect (at 45.72 67.31))
   (wire (pts (xy 27.94 144.78) (xy 29.845 144.78))
     (stroke (width 0) (type solid) (color 0 0 0 0))
@@
     (stroke (width 0) (type solid) (color 0 0 0 0))
   )
-  (wire (pts (xy 268.605 149.86) (xy 268.605 153.035))
-    (stroke (width 0) (type solid) (color 0 0 0 0))
-  )
+  (wire (pts (xy 268.605 149.86) (xy 268.605 153.67))
+    (stroke (width 0) (type solid) (color 0 0 0 0))
+  )

Commit message: Improve documentation. Generate new image. Remove irrelavant symbols in silkscreen.
Other:
- company: (none) -> jacho@mlab.cz
- title: (none) -> RFIQINT02A

Commit message: Edit UST ID
Parts:
- C1: UST_ID (none) -> 5c70984412875079b91f8867
- C10, C11, C3, C4, C5, C6, C7, C8, C9: UST_ID (none) -> 5c70984712875079b91f8b4c
- C2: UST_ID (none) -> 5c70984812875079b91f8bbf
- D1, D2: UST_ID (none) -> 5c70984512875079b91f88ac
- J3, J4, J5: UST_ID (none) -> 5c70984712875079b91f8a7b
- J6, J7: UST_ID (none) -> 5c70984712875079b91f8a7d
- L1: UST_ID (none) -> 5c70984712875079b91f8b8a
- R1: UST_ID (none) -> 5c70984512875079b91f8977
- R2, R3, R4, R5: UST_ID (none) -> 5c70984512875079b91f8979
- R6, R7: UST_ID (none) -> 5c70984512875079b91f898c
- U1: UST_ID (none) -> 5c70984712875079b91f8b82
Changed lines of the file:
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@@
+      (effects (font (size 1.27 1.27)) hide)
+    )
+    (property "UST_ID" "5c70984712875079b91f8b8a" (id 4) (at 43.815 147.32 0)
       (effects (font (size 1.27 1.27)) hide)
     )
@@
       (effects (font (size 1.27 1.27)) hide)
     )
+    (property "UST_ID" "5c70984512875079b91f8977" (id 4) (at 69.85 73.66 0)
+      (effects (font (size 1.27 1.27)) hide)
+    )
     (pin "1")
     (pin "2")
@@
       (effects (font (size 1.27 1.27)) hide)
     )
+    (property "UST_ID" "5c70984512875079b91f8979" (id 4) (at 128.27 82.55 0)
+      (effects (font (size 1.27 1.27)) hide)
+    )
     (pin "1")
     (pin "2")
@@
       (effects (font (size 1.27 1.27)) hide)
     )
+    (property "UST_ID" "5c70984512875079b91f8979" (id 4) (at 133.985 82.55 0)
+      (effects (font (size 1.27 1.27)) hide)
+    )
     (pin "1")
     (pin "2")
@@
       (effects (font (size 1.27 1.27)) hide)
     )
+    (property "UST_ID" "5c70984512875079b91f8979" (id 4) (at 139.7 82.55 0)
+      (effects (font (size 1.27 1.27)) hide)
+    )
     (pin "1")
     (pin "2")
@@
       (effects (font (size 1.27 1.27)) hide)
     )
+    (property "UST_ID" "5c70984512875079b91f8979" (id 4) (at 145.415 82.55 0)
+      (effects (font (size 1.27 1.27)) hide)
+    )
     (pin "1")
     (pin "2")
@@
       (effects (font (size 1.27 1.27)) hide)
     )
+    (property "UST_ID" "5c70984512875079b91f898c" (id 4) (at 250.19 61.595 0)
+      (effects (font (size 1.27 1.27)) hide)
+    )
     (pin "1")
     (pin "2")
@@
       (effects (font (size 1.27 1.27)) hide)
     )
+    (property "UST_ID" "5c70984512875079b91f898c" (id 4) (at 250.19 114.935 0)
+      (effects (font (size 1.27 1.27)) hide)
+    )
     (pin "1")
     (pin "2")
@@
       (effects (font (size 1.27 1.27)) hide)
     )
+    (property "UST_ID" "5c70984512875079b91f88ac" (id 4) (at 37.465 152.4 0)
+      (effects (font (size 1.27 1.27)) hide)
+    )
     (pin "1")
     (pin "2")
@@
       (effects (font (size 1.27 1.27)) hide)
     )
+    (property "UST_ID" "5c70984512875079b91f88ac" (id 4) (at 37.465 184.15 0)
+      (effects (font (size 1.27 1.27)) hide)
+    )
     (pin "1")
     (pin "2")
@@
       (effects (font (size 1.27 1.27)) hide)
     )
+    (property "UST_ID" "5c70984412875079b91f8867" (id 4) (at 46.99 184.15 0)
+      (effects (font (size 1.27 1.27)) hide)
+    )
     (pin "1")
     (pin "2")
@@
     )
     (property "Datasheet" "~" (id 3) (at 49.53 152.4 0)
+      (effects (font (size 1.27 1.27)) hide)
+    )
+    (property "UST_ID" "5c70984812875079b91f8bbf" (id 4) (at 49.53 152.4 0)
       (effects (font (size 1.27 1.27)) hide)
     )
@@
       (effects (font (size 1.27 1.27)) hide)
     )
+    (property "UST_ID" "5c70984712875079b91f8b4c" (id 4) (at 60.96 67.31 0)
+      (effects (font (size 1.27 1.27)) hide)
+    )
     (pin "1")
     (pin "2")
@@
       (effects (font (size 1.27 1.27)) hide)
     )
+    (property "UST_ID" "5c70984712875079b91f8b4c" (id 4) (at 60.96 80.01 0)
+      (effects (font (size 1.27 1.27)) hide)
+    )
     (pin "1")
     (pin "2")
@@
     )
     (property "Datasheet" "~" (id 3) (at 85.725 51.435 0)
+      (effects (font (size 1.27 1.27)) hide)
+    )
+    (property "UST_ID" "5c70984712875079b91f8b4c" (id 4) (at 85.725 51.435 0)
       (effects (font (size 1.27 1.27)) hide)
     )
@@
       (effects (font (size 1.27 1.27)) hide)
     )
+    (property "UST_ID" "5c70984712875079b91f8b4c" (id 4) (at 151.765 61.595 0)
+      (effects (font (size 1.27 1.27)) hide)
+    )
     (pin "1")
     (pin "2")
@@
       (effects (font (size 1.27 1.27)) hide)
     )
+    (property "UST_ID" "5c70984712875079b91f8b4c" (id 4) (at 151.765 67.31 0)
+      (effects (font (size 1.27 1.27)) hide)
+    )
     (pin "1")
     (pin "2")
@@
       (effects (font (size 1.27 1.27)) hide)
     )
+    (property "UST_ID" "5c70984712875079b91f8b4c" (id 4) (at 151.765 72.39 0)
+      (effects (font (size 1.27 1.27)) hide)
+    )
     (pin "1")
     (pin "2")
@@
       (effects (font (size 1.27 1.27)) hide)
     )
+    (property "UST_ID" "5c70984712875079b91f8b4c" (id 4) (at 151.765 77.47 0)
+      (effects (font (size 1.27 1.27)) hide)
+    )
     (pin "1")
     (pin "2")
@@
       (effects (font (size 1.27 1.27)) hide)
     )
+    (property "UST_ID" "5c70984712875079b91f8b4c" (id 4) (at 259.08 61.595 0)
+      (effects (font (size 1.27 1.27)) hide)
+    )
     (pin "1")
     (pin "2")
@@
       (effects (font (size 1.27 1.27)) hide)
     )
+    (property "UST_ID" "5c70984712875079b91f8b4c" (id 4) (at 259.08 114.935 0)
+      (effects (font (size 1.27 1.27)) hide)
+    )
     (pin "1")
     (pin "2")
@@
       (effects (font (size 1.524 1.524)))
     )
+    (property "UST_ID" "5c70984712875079b91f8a7b" (id 4) (at 40.64 69.85 0)
+      (effects (font (size 1.27 1.27)) hide)
+    )
     (pin "1")
     (pin "2")
@@
       (effects (font (size 1.524 1.524)))
     )
+    (property "UST_ID" "5c70984712875079b91f8a7b" (id 4) (at 196.85 41.275 0)
+      (effects (font (size 1.27 1.27)) hide)
+    )
     (pin "1")
     (pin "2")
@@
       (effects (font (size 1.524 1.524)))
     )
+    (property "UST_ID" "5c70984712875079b91f8a7b" (id 4) (at 196.85 94.615 0)
+      (effects (font (size 1.27 1.27)) hide)
+    )
     (pin "1")
     (pin "2")
@@
     (property "Datasheet" "" (id 3) (at 245.11 42.545 0)
       (effects (font (size 1.524 1.524)))
+    )
+    (property "UST_ID" "5c70984712875079b91f8a7d" (id 4) (at 245.11 42.545 0)
+      (effects (font (size 1.27 1.27)) hide)
     )
     (pin "1")
@@
       (effects (font (size 1.524 1.524)))
     )
+    (property "UST_ID" "5c70984712875079b91f8a7d" (id 4) (at 245.11 95.885 0)
+      (effects (font (size 1.27 1.27)) hide)
+    )
     (pin "1")
     (pin "10")
@@
       (effects (font (size 1.524 1.524)) hide)
     )
-    (pin "1")
+    (property "UST_ID" "5c70984712875079b91f8b82" (id 4) (at 104.14 69.85 0)
+      (effects (font (size 1.27 1.27)) hide)
+    )
+    (pin "1")
