File: hw/sch_pcb/RFIQINT02B.kicad_pcb (KiCad board)
At the start: 2 copper layers, 40.1 x 60.5 mm, 40 parts, among them J1 SATA7-67491-1030, J2 RJ45_RJHSE-5384, J3 SATA7-67491-1030, J4 SATA7-67491-1030, J5 RJ45_RJHSE-5384, J6 HEADER_2x03_PARALLEL, J7 HEADER_2x04_PARALLEL, M1 HOLE, M2 HOLE, M3 HOLE, M4 HOLE, U1 Si53322

Commit message: #5
Parts:
- added C15: 100nF, Mlab_R:SMD-0805, B.Cu at (57.4, -26.5)
- added C16: 100nF, Mlab_R:SMD-0805, B.Cu at (53.2, -26.5)
- added C17: 100nF, Mlab_R:SMD-0805, B.Cu at (49.0, -23.9)
- added R12: 1k, Mlab_R:SMD-0805, B.Cu at (53.2, -23.9)
- added R13: 1k, Mlab_R:SMD-0805, B.Cu at (49.0, -26.5)
- added R14: 1k, Mlab_R:SMD-0805, B.Cu at (57.4, -23.9)
Connections:
- J1 pad 1: GND -> Net-(J1-Pad1)
- J1 pad 4: GND -> Net-(J1-Pad1)
- J1 pad 7: GND -> Net-(J1-Pad1)
- J3 pad 1: GND -> Net-(J3-Pad1)
- J3 pad 4: GND -> Net-(J3-Pad1)
- J3 pad 7: GND -> Net-(J3-Pad1)
- J4 pad 1: GND -> Net-(J4-Pad1)
- J4 pad 4: GND -> Net-(J4-Pad1)
- J4 pad 7: GND -> Net-(J4-Pad1)

Commit message: #6 #5
Parts:
- C1, C10, C11, C12, C15, C16, C17, C3, C4, C5, C6, C7, C8, C9, L1, R1, R10, R11, R12, R13, R14, R2, R3, R4, R5, R6, R7, R8, R9: footprint Mlab_R:SMD-0805 -> Resistor_SMD:R_0805_2012Metric
- C13, C2: footprint Mlab_R:SMD-0805 -> Capacitor_SMD:C_0805_2012Metric
- C14: footprint Mlab_C:TantalC_SizeC_Reflow -> Capacitor_Tantalum_SMD:CP_EIA-7132-28_AVX-C
- D1, D2: footprint Mlab_D:Diode-SMA_Standard -> Diode_SMD:D_SMA
- moved M3 144.8 mm to (35.6, -55.9)
- moved M1 107.9 mm to (35.6, -5.08)
- moved C16 45.9 mm to (13.9, -50.3), turned to -90 degrees
- moved R14 45.4 mm to (13.6, -11.7), turned to 90 degrees
- moved R13 44.6 mm to (11.3, -50.3), turned to -90 degrees
- moved C15 41.5 mm to (18.0, -39.7), turned to -90 degrees
- moved R12 36.4 mm to (20.4, -39.7), turned to -90 degrees
- moved C17 35.5 mm to (15.6, -11.7), turned to 90 degrees
- moved C9 0.18 mm to (21.7, -23.6)
- moved C6 0.18 mm to (21.7, -30.8)
- moved M4 0.11 mm to (5.08, -55.9)
- moved R8 0.09 mm to (18.9, -22.9)
Routing:
- net Net-(J4-Pad1): track 0.00 -> 14.6 mm, vias 0 -> 1
- net Net-(J1-Pad1): track 0.00 -> 14.3 mm, vias 0 -> 1
- net Net-(J3-Pad1): track 0.00 -> 13.8 mm, vias 0 -> 1
- net +3V8: track 46.7 -> 44.9 mm
Other:
- board text added: "MLAB.CZ RFIQINT02B"
