File: hw/sch_pcb/RFIQINT02B.kicad_sch (KiCad schematic)
At the start: 40 parts, among them J1 SATA7-67491-1030, J2 RJ45_RJHSE-5384, J3 SATA7-67491-1030, J4 SATA7-67491-1030, J5 RJ45_RJHSE-5384, J6 HEADER_2x03_PARALLEL, J7 HEADER_2x04_PARALLEL, M1 HOLE, M2 HOLE, M3 HOLE, M4 HOLE, U1 Si53322

Commit message: #5
Parts:
- added C15, C16, C17: 100nF, Mlab_R:SMD-0805, symbol Device:C
- added R12, R13, R14: 1k, Mlab_R:SMD-0805, symbol Device:R
Connections:
- net GND: now also C15.2, C16.2, C17.2, R12.2, R13.2, R14.2; no longer J1.1, J1.4, J1.7, J3.1, J3.4, J3.7, J4.1, J4.4, J4.7
- new net: C17.1, J1.1, J1.4, J1.7, R14.1
- new net: C16.1, J4.1, J4.4, J4.7, R13.1
- new net: C15.1, J3.1, J3.4, J3.7, R12.1

Commit message: #6 #5
Parts:
- C1, C10, C11, C12, C15, C16, C17, C3, C4, C5, C6, C7, C8, C9, L1, R1, R10, R11, R12, R13, R14, R2, R3, R4, R5, R6, R7, R8, R9: footprint Mlab_R:SMD-0805 -> Resistor_SMD:R_0805_2012Metric
- C13, C2: footprint Mlab_R:SMD-0805 -> Capacitor_SMD:C_0805_2012Metric
- C14: footprint Mlab_C:TantalC_SizeC_Reflow -> Capacitor_Tantalum_SMD:CP_EIA-7132-28_AVX-C
- D1, D2: footprint Mlab_D:Diode-SMA_Standard -> Diode_SMD:D_SMA
